Commit message: lidar model, no sim

File: description/gazebo_control.xacro (robot description, xacro)
@@ -12,4 +12,9 @@
             <topic>cmd_vel</topic>
         </plugin>
+        <plugin
+      filename="libignition-gazebo-sensors-system.so"
+      name="ignition::gazebo::systems::Sensors">
+      <render_engine>ogre2</render_engine>
+    </plugin>
     </gazebo>
 </robot>

File: description/materials.xacro (robot description, xacro)
@@ -13,3 +13,9 @@
         <color rgba="0 0 0 1" />
     </material>
+    <material name="red">
+        <color rgba="1 0 0 1" />
+    </material>
+    <material name="green">
+        <color rgba="0 1 0 1" />
+    </material>
 </robot>

File: description/robot.urdf (robot description, URDF)
Before this commit: robot robot, 5 links, 4 joints
Links:
- added link laser_link, mass 0.1; collision cylinder length=0.04 radius=0.05; visual cylinder length=0.04 radius=0.05
Joints:
- added joint laser_joint: type fixed, parent chassis_link, child laser_link, origin xyz=0.1 0 0.175 rpy=0 0 0

File: description/robot.urdf.xacro (robot description, xacro)
@@ -3,5 +3,7 @@
     <!-- CHASSIS AND WHEELS -->
     <xacro:include filename="robot_core.xacro" />
-    <!-- TELEOP SIMULATION -->
+    <!-- LiDAR-->
+    <xacro:include filename="lidar.xacro" />
+    <!-- DIFF_DRIVE SIMULATION -->
     <xacro:include filename="gazebo_control.xacro" />
 </robot>

Commit message: Lidar sim / switch to gazebo-classic

File: description/gazebo_control.xacro (robot description, xacro)
@@ -2,19 +2,20 @@
 <robot xmlns:xacro="http://www.ros.org/wiki/xacro" >
     <gazebo>
-        <plugin filename="libignition-gazebo-diff-drive-system.so" name="ignition::gazebo::systems::DiffDrive" >
-            <!-- WHEEL INFO -->
+        <plugin name="diff_drive" filename="libgazebo_ros_diff_drive.so">
+            <!-- Wheel Information -->
             <left_joint>left_wheel_joint</left_joint>
             <right_joint>right_wheel_joint</right_joint>
-            <wheel_seperation>0.35</wheel_seperation>
-            <wheel_radius>0.05</wheel_radius>
-            <!-- I/O -->
-            <odom_publish_frequency>1</odom_publish_frequency>
-            <topic>cmd_vel</topic>
+            <wheel_separation>0.35</wheel_separation>
+            <wheel_diameter>0.1</wheel_diameter>
+            <!-- Limits -->
+            <max_wheel_torque>200</max_wheel_torque>
+            <max_wheel_acceleration>10.0</max_wheel_acceleration>
+            <!-- Output -->
+            <odometry_frame>odom</odometry_frame>
+            <robot_base_frame>base_link</robot_base_frame>
+            <publish_odom>true</publish_odom>
+            <publish_odom_tf>true</publish_odom_tf>
+            <publish_wheel_tf>true</publish_wheel_tf>
         </plugin>
-        <plugin
-      filename="libignition-gazebo-sensors-system.so"
-      name="ignition::gazebo::systems::Sensors">
-      <render_engine>ogre2</render_engine>
-    </plugin>
     </gazebo>
 </robot>

File: description/lidar.xacro (robot description, xacro)
@@ -4,55 +4,50 @@
     <joint name="laser_joint" type="fixed">
         <parent link="chassis_link" />
-        <child link="laser_link" />
+        <child link="laser_frame" />
         <origin xyz="0.1 0 0.175" rpy="0 0 0" />
     </joint>
-    <link name="laser_link">
+    <link name="laser_frame">
         <visual>
             <geometry>
-                <cylinder radius="0.05" length="0.04" />
+                <cylinder radius="0.05" length="0.04"/>
             </geometry>
-            <material name="red" />
+            <material name="red"/>
         </visual>
         <collision>
             <geometry>
-                <cylinder radius="0.05" length="0.04" />
+                <cylinder radius="0.05" length="0.04"/>
             </geometry>
         </collision>
-        <xacro:inertial_cylinder mass="0.1" length="0.4" radius="0.5">
-            <origin xyz="0 0 0" rpy="0 0 0" />
+        <xacro:inertial_cylinder mass="0.1" length="0.04" radius="0.05">
+            <origin xyz="0 0 0" rpy="0 0 0"/>
         </xacro:inertial_cylinder>
     </link>
-    <frame name="laser_frame" attached_to='laser_link'>
-        <pose>0 0 0 0 0 0</pose>
-    </frame>
     <gazebo reference="laser_frame">
-        <sensor name='gpu_lidar' type='gpu_lidar'>
-            <pose>0 0 0 0 0 0</pose>
-    <topic>lidar</topic>
-    <update_rate>10</update_rate>
-    <ray>
-        <scan>
-            <horizontal>
-                <samples>640</samples>
-                <resolution>1</resolution>
-                <min_angle>-1.396263</min_angle>
-                <max_angle>1.396263</max_angle>
-            </horizontal>
-            <vertical>
-                <samples>1</samples>
-                <resolution>0.01</resolution>
-                <min_angle>0</min_angle>
-                <max_angle>0</max_angle>
-            </vertical>
-        </scan>
-        <range>
-            <min>0.08</min>
-            <max>10.0</max>
-            <resolution>0.01</resolution>
-        </range>
-    </ray>
-    <always_on>1</always_on>
-    <visualize>true</visualize>
-</sensor>
+        <material>Gazebo/Red</material>
+        <sensor name="laser" type="ray">
+            <pose> 0 0 0 0 0 0 </pose>
+            <visualize>true</visualize>
+            <update_rate>10</update_rate>
+            <ray>
+                <scan>
+                    <horizontal>
+                        <samples>360</samples>
+                        <min_angle>-3.14</min_angle>
+                        <max_angle>3.14</max_angle>
+                    </horizontal>
+                </scan>
+                <range>
+                    <min>0.3</min>
+                    <max>12</max>
+                </range>
+            </ray>
+            <plugin name="laser_controller" filename="libgazebo_ros_ray_sensor.so">
+                <ros>
+                    <argument>~/out:=scan</argument>
+                </ros>
+                <output_type>sensor_msgs/LaserScan</output_type>
+                <frame_name>laser_frame</frame_name>
+            </plugin>
+        </sensor>
     </gazebo>
 </robot>

File: description/robot.urdf.xacro (robot description, xacro)
@@ -5,4 +5,6 @@
     <!-- LiDAR-->
     <xacro:include filename="lidar.xacro" />
+    <!-- CAMERA -->
+    <xacro:include filename="camera.xacro" />
     <!-- DIFF_DRIVE SIMULATION -->
     <xacro:include filename="gazebo_control.xacro" />

File: description/robot_core.xacro (robot description, xacro)
@@ -30,4 +30,7 @@
         </xacro:inertial_box>
     </link>
+    <gazebo reference="chassis_link">
+        <material>Gazebo/White</material>
+    </gazebo>
     <!-- LEFT WHEEL LINK -->
     <joint name="left_wheel_joint" type="continuous">
@@ -53,4 +56,7 @@
         </xacro:inertial_cylinder>
     </link>
+    <gazebo reference="left_wheel_link">
+        <material>Gazebo/Blue</material>
+    </gazebo>
     <!-- RIGHT WHEEL LINK -->
     <joint name="right_wheel_joint" type="continuous">
@@ -76,4 +82,7 @@
         </xacro:inertial_cylinder>
     </link>
+    <gazebo reference="right_wheel_link">
+        <material>Gazebo/Blue</material>
+    </gazebo>
     <!-- CASTER WHEEL LINK -->
     <joint name="caster_wheel_joint" type="fixed">
@@ -98,5 +107,6 @@
         </xacro:inertial_sphere>
     </link>
-    <gazebo reference="caster_wheel">
+    <gazebo reference="caster_wheel_link">
+        <material>Gazebo/Black</material>
         <mu1 value="0.001"/>
         <mu2 value="0.001"/>
