Commit message: dual cameras

File: description/camera.xacro (robot description, xacro)
@@ -1,27 +1,27 @@
 <?xml version="1.0"?>
 <robot xmlns:xacro="http://www.ros.org/wiki/xacro" >
-    <!-- CAMERA -->
-    <joint name="camera_joint" type="fixed">
+    <!-- RIGHT CAMERA -->
+    <joint name="right_camera_joint" type="fixed">
         <parent link="chassis_link" />
-        <child link="camera_link" />
-        <origin xyz="0.305 0 0.08" rpy="0 0 0" />
+        <child link="right_camera_link" />
+        <origin xyz="0.305 -0.12 0.08" rpy="0 0 0" />
     </joint>
-    <link name="camera_link">
+    <link name="right_camera_link">
         <visual>
             <geometry>
                 <box size="0.010 0.03 0.03" />
             </geometry>
-            <material name="green"/>
+            <material name="red"/>
         </visual>
     </link>
-    <joint name="camera_optical_joint" type="fixed">
-        <parent link="camera_link" />
-        <child link="camera_link_optical" />
+    <joint name="right_camera_optical_joint" type="fixed">
+        <parent link="right_camera_link" />
+        <child link="right_camera_link_optical" />
         <origin xyz="0 0 0" rpy="-${pi/2} 0 -${pi/2}" />
     </joint>
-    <link name="camera_link_optical"></link>
-    <gazebo reference="camera_link">
-        <material>Gazebo/Green</material>
-        <sensor name="camera" type="camera">
+    <link name="right_camera_link_optical"></link>
+    <gazebo reference="right_camera_link">
+        <material>Gazebo/Red</material>
+        <sensor name="right_camera" type="camera">
             <pose> 0 0 0 0 0 0 </pose>
             <visualize>false</visualize>
@@ -39,6 +39,49 @@
                 </clip>
             </camera>
-            <plugin name="camera_controller" filename="libgazebo_ros_camera.so">
-                <frame_name>camera_link_optical</frame_name>
+            <plugin name="right_camera_controller" filename="libgazebo_ros_camera.so">
+                <frame_name>right_camera_link_optical</frame_name>
+            </plugin>
+        </sensor>
+    </gazebo>
+    <!-- LEFT CAMERA -->
+    <joint name="left_camera_joint" type="fixed">
+        <parent link="chassis_link" />
+        <child link="left_camera_link" />
+        <origin xyz="0.305 0.12 0.08" rpy="0 0 0" />
+    </joint>
+    <link name="left_camera_link">
+        <visual>
+            <geometry>
+                <box size="0.010 0.03 0.03" />
+            </geometry>
+            <material name="green"/>
+        </visual>
+    </link>
+    <joint name="left_camera_optical_joint" type="fixed">
+        <parent link="left_camera_link" />
+        <child link="left_camera_link_optical" />
+        <origin xyz="0 0 0" rpy="-${pi/2} 0 -${pi/2}" />
+    </joint>
+    <link name="left_camera_link_optical"></link>
+    <gazebo reference="left_camera_link">
+        <material>Gazebo/Green</material>
+        <sensor name="left_camera" type="camera">
+            <pose> 0 0 0 0 0 0 </pose>
+            <visualize>false</visualize>
+            <update_rate>10</update_rate>
+            <camera>
+                <horizontal_fov>1.089</horizontal_fov>
+                <image>
+                    <format>R8G8B8</format>
+                    <width>640</width>
+                    <height>480</height>
+                </image>
+                <clip>
+                    <near>0.05</near>
+                    <far>8.0</far>
+                </clip>
+            </camera>
+            <plugin name="left_camera_controller" filename="libgazebo_ros_camera.so">
+                <frame_name>left_camera_link_optical</frame_name>
             </plugin>
         </sensor>
