Commit message: ros2 control tweaks / rvis config

File: description/robot.urdf.xacro (robot description, xacro)
@@ -1,4 +1,5 @@
 <?xml version="1.0"?>
 <robot xmlns:xacro="http://www.ros.org/wiki/xacro"  name="robot">
+    <xacro:arg name="use_ros2_control" default="true" />
     <!-- CHASSIS AND WHEELS -->
     <xacro:include filename="robot_core.xacro" />
@@ -8,5 +9,9 @@
     <xacro:include filename="camera.xacro" />
     <!-- CONTROL -->
-    <!-- <xacro:include filename="gazebo_control.xacro" /> -->
-    <xacro:include filename="ros2_control.xacro" />
+    <xacro:if value="$(arg use_ros2_control)" >
+        <xacro:include filename="ros2_control.xacro" />
+    </xacro:if>
+    <xacro:unless value="$(arg use_ros2_control)" >
+        <xacro:include filename="gazebo_control.xacro" />
+    </xacro:unless>
 </robot>

File: description/robot_core.xacro (robot description, xacro)
@@ -49,5 +49,5 @@
         <collision>
             <geometry>
-                <cylinder radius="0.05" length="0.04" />
+                <sphere radius="0.05" />
             </geometry>
         </collision>
@@ -75,5 +75,5 @@
         <collision>
             <geometry>
-                <cylinder radius="0.05" length="0.04" />
+                <sphere radius="0.05" />
             </geometry>
         </collision>

Commit message: 3d velodyne lidar sim

File: description/robot.urdf.xacro (robot description, xacro)
@@ -2,8 +2,14 @@
 <robot xmlns:xacro="http://www.ros.org/wiki/xacro"  name="robot">
     <xacro:arg name="use_ros2_control" default="true" />
+    <xacro:arg name="gpu" default="false"/>
+    <xacro:property name="gpu" value="$(arg gpu)" />
     <!-- CHASSIS AND WHEELS -->
     <xacro:include filename="robot_core.xacro" />
     <!-- LiDAR-->
-    <xacro:include filename="lidar.xacro" />
+    <!-- <xacro:include filename="lidar.xacro" /> -->
+    <xacro:include filename="VLP-16.xacro"/>
+    <xacro:VLP-16 parent="chassis_link" name="velodyne" topic="/velodyne_points" hz="10" samples="440" gpu="${gpu}">
+      <origin xyz="0.1 0 0.15" rpy="0 0 0" />
+    </xacro:VLP-16>
     <!-- CAMERA -->
     <xacro:include filename="camera.xacro" />
